Commit message: Various manual fixes to get it to render nicely. Left back wheel frame is off, hacked it in place (ish)

File: ROS/osr_description/urdf/osr_description.urdf (robot description, URDF)
Before this commit: robot osr_description, 15 links, 13 joints
Joints:
- removed joint body_axis
- added joint body_axis_left: type continuous, parent base_link, child left_rocker, origin xyz=-0.263500464134776 0.18018125 0.225295670634321 rpy=-1.53745923062483 0 -1.5707963267949, axis 0 0 1
- added joint body_axis_right: type continuous, parent base_link, child right_rocker, origin xyz=-0.2635 -0.14208 0.2253 rpy=-1.5375 0 -1.5708, axis 0 0 1, limit lower=0 upper=0 effort=0 velocity=0
- joint back_left_corner_joint: axis 0 1 0 -> 0 0 1; origin xyz=0.01905 0.068201 -0.05715 rpy=-1.5708 1.5708 0 -> xyz=0.01905 0.068201 -0.05715 rpy=0 1.5708 0; type revolute -> continuous
- joint back_left_drive_joint: axis 1 0 0 -> 0 0 1; origin xyz=0 0.066549 0 rpy=1.5708 1.5708 0 -> xyz=0 0.2705 0 rpy=1.5708 1.5708 0
- joint back_right_corner_joint: axis 0 0 0 -> 0 0 1; origin xyz=0.0381 0.088265 -0.0762 rpy=-1.5708 -1.5708 0 -> xyz=0.0381 0.088265 -0.0762 rpy=0 -1.5708 0; type revolute -> continuous
- joint back_right_drive_joint: axis 0 0 0 -> 0 0 1
- joint front_left_corner_joint: axis 0 0 0 -> 0 0 1; type revolute -> continuous
- joint front_left_drive_joint: axis 0 0 0 -> 0 0 1
- joint front_right_corner_joint: axis 0 0 0 -> 0 0 1; type revolute -> continuous
- joint front_right_drive_joint: axis 0 0 0 -> 0 0 1
- joint left_lb_axis: axis 0 0 0 -> 0 0 1; type revolute -> continuous
- joint middle_left_drive_joint: axis 0 0 0 -> 0 0 1
- joint right_middle_drive_joint: axis 0 0 0 -> 0 0 1
- joint right_rb_axis: axis 0 0 0 -> 0 0 1; type revolute -> continuous
